File: hardware/robot-mainboard/adr1-robot.kicad_sch (KiCad schematic)
At the start: 41 parts, among them J1 SMA_868MHz, J2 SMA_GNSS, J3 USB-C (Debug/FW Update), J4 SWD Debug, J5 CAN Bus (CANH,CANL,+24V,GND), J6 RS485 (A,B,+12V,GND), J7 Motor CAN + Power, J8 microSD, U1 STM32H743VIT6, U10 ADS1115 (0x48)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

Commit message: fix: Upgrade all ICs to industrial grade (-40°C to +85°C minimum)
Replace 9 components that failed industrial temperature grade audit:

- IS42S16400J-7TL → IS42S16400J-7TLI (Industrial SDRAM)
- HC-SR04 → MaxBotix MB1240 XL-MaxSonar-EZ4 (Industrial IP67, -40/+85°C)
- OV5640-AF → onsemi AR0234CS (Automotive -40/+105°C, 2.3MP global shutter)
- TFmini-S → TFmini-S-I (Industrial version, -40/+65°C, IP65)
- E6B2-CWZ6C → ams AS5047P (AEC-Q100, -40/+125°C, magnetic encoder)
- XL4015 → TI TPS54360BDDAR (Industrial buck, -40/+150°C Tj)
- ILI9488 MSP3520 → Newhaven NHD-3.5-320240MF-ATXI (Industrial -30/+80°C)
- TP4056 → Removed (redundant with MCP73871-2CCI)
- WS2812B-2020 → APA102-2020 (Industrial -40/+85°C, SPI interface)

Updated across: BOM, KiCad schematics, KiCad PCBs, circuit diagrams,
sensor documentation, and firmware drivers (ultrasonic + LED).

Total project cost impact: ₹131,585 → ₹143,623 (+9.2% for full industrial grade)

https://claude.ai/code/session_01JEQm9q7KiSgXTYN94pugrd
Parts:
- added U19: IS42S16400J-7TLI (Industrial), Package_SO:TSOP-II-54_22.2x10.16mm_P0.8mm, symbol Memory_RAM:IS42S16400J
- added U20: TPS54360BDDAR (24V→12V) Industrial, Package_SO:HSOP-8-1EP_3.9x4.9mm_P1.27mm, symbol Regulator_Switching:TPS54360B
- U14: value W25Q128JVSIQ -> W25Q128JVSIQ (Industrial)
- U15: value LM2596S-5.0 (24V→5V) -> LM2596S-5.0 (24V→5V) Industrial
Changed lines of the file:
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@@
   )
   ;; ═══════════════════════════════════════════════════════════════
-  ;; QSPI FLASH - W25Q128
+  ;; QSPI FLASH - W25Q128 Industrial (-40°C to +85°C)
   ;; ═══════════════════════════════════════════════════════════════
   (symbol (lib_id "Memory_Flash:W25Q128JVS") (at 203.2 76.2 0) (unit 1)
@@
     (uuid "flash-w25q128")
     (property "Reference" "U14" (at 203.2 63.5 0) (effects (font (size 1.27 1.27))))
-    (property "Value" "W25Q128JVSIQ" (at 203.2 66.04 0) (effects (font (size 1.27 1.27))))
+    (property "Value" "W25Q128JVSIQ (Industrial)" (at 203.2 66.04 0) (effects (font (size 1.27 1.27))))
     (property "Footprint" "Package_SO:SOIC-8_5.23x5.23mm_P1.27mm" (at 203.2 68.58 0) (effects (font (size 1.27 1.27)) hide))
   )
   ;; ═══════════════════════════════════════════════════════════════
-  ;; POWER SUPPLY - LM2596 (24V→5V)
+  ;; SDRAM - IS42S16400J Industrial (-40°C to +85°C)
+  ;; ═══════════════════════════════════════════════════════════════
+  (symbol (lib_id "Memory_RAM:IS42S16400J") (at 203.2 101.6 0) (unit 1)
+    (in_bom yes) (on_board yes) (dnp no)
+    (uuid "sdram-is42s16400j")
+    (property "Reference" "U19" (at 203.2 88.9 0) (effects (font (size 1.27 1.27))))
+    (property "Value" "IS42S16400J-7TLI (Industrial)" (at 203.2 91.44 0) (effects (font (size 1.27 1.27))))
+    (property "Footprint" "Package_SO:TSOP-II-54_22.2x10.16mm_P0.8mm" (at 203.2 93.98 0) (effects (font (size 1.27 1.27)) hide))
+  )
+  ;; ═══════════════════════════════════════════════════════════════
+  ;; POWER SUPPLY - LM2596S (24V→5V) Industrial (-40°C to +125°C Tj)
   ;; ═══════════════════════════════════════════════════════════════
   (symbol (lib_id "Regulator_Switching:LM2596S-5") (at 50.8 279.4 0) (unit 1)
@@
     (uuid "buck-5v")
     (property "Reference" "U15" (at 50.8 266.7 0) (effects (font (size 1.27 1.27))))
-    (property "Value" "LM2596S-5.0 (24V→5V)" (at 50.8 269.24 0) (effects (font (size 1.27 1.27))))
+    (property "Value" "LM2596S-5.0 (24V→5V) Industrial" (at 50.8 269.24 0) (effects (font (size 1.27 1.27))))
     (property "Footprint" "Package_TO_SOT_SMD:TO-263-5_TabPin3" (at 50.8 271.78 0) (effects (font (size 1.27 1.27)) hide))
   )
@@
   ;; TEXT ANNOTATIONS (Net Labels)
   ;; ═══════════════════════════════════════════════════════════════
+  ;; ═══════════════════════════════════════════════════════════════
+  ;; POWER SUPPLY - TPS54360B (24V→12V) Industrial (-40°C to +150°C Tj)
+  ;; ═══════════════════════════════════════════════════════════════
+  (symbol (lib_id "Regulator_Switching:TPS54360B") (at 152.4 279.4 0) (unit 1)
+    (in_bom yes) (on_board yes) (dnp no)
+    (uuid "buck-12v")
+    (property "Reference" "U20" (at 152.4 266.7 0) (effects (font (size 1.27 1.27))))
+    (property "Value" "TPS54360BDDAR (24V→12V) Industrial" (at 152.4 269.24 0) (effects (font (size 1.27 1.27))))
+    (property "Footprint" "Package_SO:HSOP-8-1EP_3.9x4.9mm_P1.27mm" (at 152.4 271.78 0) (effects (font (size 1.27 1.27)) hide))
+  )
   (text "POWER SUPPLY SECTION" (at 50.8 254.0 0) (effects (font (size 2.54 2.54) bold)))
   (text "MCU SECTION" (at 152.4 38.1 0) (effects (font (size 2.54 2.54) bold)))
